File: kicad/hip-factor-3-l/hip-factor-3-l.kicad_pcb (KiCad board)
At the start: 2 copper layers, 175.3 x 92 mm, 72 parts, among them J1 Conn_01x12_Female, J2 Conn_01x12_Female, J3 AudioJack4, SW1 SW_Push, SW10 SW_Push, SW11 SW_Push, SW12 SW_Push, SW13 SW_Push, SW14 SW_Push, SW15 SW_Push, SW16 SW_Push, SW17 SW_Push, SW18 SW_Push, SW19 SW_Push, SW2 SW_Push, SW20 SW_Push, SW21 SW_Push, SW22 SW_Push, SW23 SW_Push, SW24 SW_Push, SW25 SW_Push, SW26 SW_Push, SW27 SW_Push, SW28 SW_Push, SW29 SW_Push, SW3 SW_Push, SW30 SW_Push, SW31 SW_Push, SW32 SW_Push, SW33 SW_Push, SW34 SW_Push, SW35 SW_Push, SW4 SW_Push, SW5 SW_Push, SW6 SW_Push, SW7 SW_Push, SW8 SW_Push, SW9 SW_Push

Commit message: update pcb and case
Parts:
- D1, D10, D11, D12, D13, D14, D15, D16, D17, D18, D19, D2, D20, D21, D22, D23, D24, D25, D26, D27, D28, D29, D3, D30, D31, D32, D33, D34, D4, D5, D6, D7, D8, D9: footprint Diode_SMD:D_SOD-123 -> wyatt:D_SOD-123_or_short
- J3: footprint Connector_Audio:Jack_3.5mm_PJ320E_Horizontal -> wyatt:Jack_3.5mm_PJ320A_Horizontal
- SW35: footprint Button_Switch_SMD:SW_SPST_PTS645 -> Button_Switch_SMD:SW_SPST_TL3342
- moved D33 4.75 mm to (160.0, 116.0)
- moved D34 4.75 mm to (188.5, 116.0)
- moved SW33 4.75 mm to (149.9, 113.5)
- moved SW34 4.75 mm to (178.4, 113.5)
- moved J1 2.54 mm to (203.2, 35.6)
- moved J3 1.92 mm to (193.9, 89.9)
- moved SW35 1.27 mm to (195.6, 40.6)
Routing:
- net /res: track 14.7 -> 12.0 mm
- net /row4: track 202.6 -> 200.1 mm
- net /row1: track 169.6 -> 167.0 mm
- net /row3: track 186.8 -> 184.3 mm
- net /row2: track 187.3 -> 184.8 mm
- net +5V: track 50.0 -> 52.0 mm
- net /col6: track 131.2 -> 129.3 mm
- net /row5: track 217.2 -> 215.4 mm
- net /col7: track 105.7 -> 107.4 mm
Other:
- board size 175.3 x 92 mm -> 172.7 x 92 mm
