File: kicad/hip-factor-3-r/hip-factor-3-r.kicad_pcb (KiCad board)
At the start: 2 copper layers, 182.1 x 92 mm, 72 parts, among them J1 Conn_01x12_Female, J2 Conn_01x12_Female, J3 AudioJack4, SW1 SW_Push, SW10 SW_Push, SW11 SW_Push, SW12 SW_Push, SW13 SW_Push, SW14 SW_Push, SW15 SW_Push, SW16 SW_Push, SW17 SW_Push, SW18 SW_Push, SW19 SW_Push, SW2 SW_Push, SW20 SW_Push, SW21 SW_Push, SW22 SW_Push, SW23 SW_Push, SW24 SW_Push, SW25 SW_Push, SW26 SW_Push, SW27 SW_Push, SW28 SW_Push, SW29 SW_Push, SW3 SW_Push, SW30 SW_Push, SW31 SW_Push, SW32 SW_Push, SW33 SW_Push, SW34 SW_Push, SW36 SW_Push, SW4 SW_Push, SW5 SW_Push, SW6 SW_Push, SW7 SW_Push, SW8 SW_Push, SW9 SW_Push

Commit message: update pcb and case
Parts:
- D1, D10, D11, D12, D13, D14, D15, D16, D17, D18, D19, D2, D20, D21, D22, D23, D24, D25, D26, D27, D28, D29, D3, D30, D31, D32, D33, D34, D4, D5, D6, D7, D8, D9: footprint Diode_SMD:D_SOD-123 -> wyatt:D_SOD-123_or_short
- J3: footprint Connector_Audio:Jack_3.5mm_PJ320E_Horizontal -> wyatt:Jack_3.5mm_PJ320A_Horizontal
- SW36: footprint Button_Switch_SMD:SW_SPST_PTS645 -> Button_Switch_SMD:SW_SPST_TL3342
- moved D29 4.75 mm to (42.5, 116.0)
- moved D30 4.75 mm to (71.0, 116.0)
- moved SW29 4.75 mm to (52.6, 118.5)
- moved SW30 4.75 mm to (81.1, 118.5)
- moved J2 2.54 mm to (27.9, 35.6)
- moved J3 2.02 mm to (37.2, 85.3)
- moved SW36 1.60 mm to (35.6, 40.6)
Routing:
- net /row5: track 228.8 -> 242.9 mm
- net /col1: track 115.3 -> 120.1 mm
- net /row4: track 242.4 -> 239.9 mm
- net /row3: track 190.4 -> 187.8 mm
- net /row2: track 202.3 -> 199.8 mm
- net /row1: track 188.4 -> 185.9 mm
- net /res: track 14.4 -> 12.0 mm
- net /col2: track 134.5 -> 136.4 mm
Other:
- board size 182.1 x 92 mm -> 179.6 x 92 mm
